File: Franzininho Wearable/FrontEnd.sch (KiCad schematic (older format))
At the start: 11 parts, among them U2 LM324N_NOPB

Commit message: Correção das bibliotecas de simbolos
Parts:
- removed C1: 47u, symbol Franzininho-Wearable-rescue:C_Small-Device
- removed C5: 100n, symbol Franzininho-Wearable-rescue:C_Small-Device
- removed R1: 82k, symbol Franzininho-Wearable-rescue:R_US-Device
- removed R2, R7, R8: 100k, symbol Franzininho-Wearable-rescue:R_US-Device
- removed R3: 1k, symbol Franzininho-Wearable-rescue:R_US-Device
- removed R4: 10k, symbol Franzininho-Wearable-rescue:R_US-Device
- removed R5: 1M, symbol Franzininho-Wearable-rescue:R_US-Device
- removed R6: 80k, symbol Franzininho-Wearable-rescue:R_US-Device
- added C5: 47u, symbol Device:C
- added C6: 100n, symbol Device:C
- added R1, R6: 82k, symbol Device:R
- added R2, R7, R8: 100k, symbol Device:R
- added R3: 1k, symbol Device:R
- added R4: 10k, symbol Device:R
- added R5: 1M, symbol Device:R
- U2: symbol Franzininho-Wearable-rescue:LM324N_NOPB-LM324N_NOPB -> Franzininho_Wearable_SchLib:LM324N_NOPB
- U2: symbol LM324N_NOPB:LM324N_NOPB -> Franzininho_Wearable_SchLib:LM324N_NOPB
Changed lines of the file:
@@
 $EndDescr
 $Comp
-L Franzininho-Wearable-rescue:LM324N_NOPB-LM324N_NOPB U?
+L Franzininho_Wearable_SchLib:LM324N_NOPB U?
 U 4 1 610191DF
 P 5950 5750
@@
 	1    0    0    -1
 $EndComp
-$Comp
-L Franzininho-Wearable-rescue:R_US-Device R?
-U 1 1 61019213
-P 6800 5750
-AR Path="/61019213" Ref="R?"  Part="1"
-AR Path="/6100EEBD/61019213" Ref="R8"  Part="1"
-F 0 "R8" V 6595 5750 50  0000 C CNN
-F 1 "100k" V 6686 5750 50  0000 C CNN
-F 2 "" V 6840 5740 50  0001 C CNN
-F 3 "~" H 6800 5750 50  0001 C CNN
-	1    6800 5750
-	0    1    1    0
-$EndComp
 Wire Wire Line
 	6650 5750 6450 5750
@@
 +BATT
 $Comp
-L LM324N_NOPB:LM324N_NOPB U?
+L Franzininho_Wearable_SchLib:LM324N_NOPB U?
 U 2 1 61019251
 P 7100 2400
@@
 	5500 2600 5500 2900
 $Comp
-L LM324N_NOPB:LM324N_NOPB U?
+L Franzininho_Wearable_SchLib:LM324N_NOPB U?
 U 1 1 610191F9
 P 5500 2300
@@
 Wire Wire Line
 	5950 2300 5950 1600
-$Comp
-L Franzininho-Wearable-rescue:R_US-Device R?
-U 1 1 610191CD
-P 5450 1600
-AR Path="/610191CD" Ref="R?"  Part="1"
-AR Path="/6100EEBD/610191CD" Ref="R4"  Part="1"
-F 0 "R4" V 5245 1600 50  0000 C CNN
-F 1 "10k" V 5336 1600 50  0000 C CNN
-F 2 "" V 5490 1590 50  0001 C CNN
-F 3 "~" H 5450 1600 50  0001 C CNN
-	1    5450 1600
-	0    1    1    0
-$EndComp
-$Comp
-L Franzininho-Wearable-rescue:R_US-Device R?
-U 1 1 610191C7
-P 4850 2200
-AR Path="/610191C7" Ref="R?"  Part="1"
-AR Path="/6100EEBD/610191C7" Ref="R1"  Part="1"
-F 0 "R1" V 4645 2200 50  0000 C CNN
-F 1 "82k" V 4736 2200 50  0000 C CNN
-F 2 "" V 4890 2190 50  0001 C CNN
-F 3 "~" H 4850 2200 50  0001 C CNN
-	1    4850 2200
-	0    1    1    0
-$EndComp
-$Comp
-L Franzininho-Wearable-rescue:R_US-Device R?
-U 1 1 610191C1
-P 4850 2400
-AR Path="/610191C1" Ref="R?"  Part="1"
-AR Path="/6100EEBD/610191C1" Ref="R2"  Part="1"
-F 0 "R2" V 4950 2400 50  0000 C CNN
-F 1 "100k" V 5050 2400 50  0000 C CNN
-F 2 "" V 4890 2390 50  0001 C CNN
-F 3 "~" H 4850 2400 50  0001 C CNN
-	1    4850 2400
-	0    1    1    0
-$EndComp
 Wire Wire Line
 	6250 2300 5950 2300
@@
 Wire Wire Line
 	6550 2300 6700 2300
-$Comp
-L Franzininho-Wearable-rescue:R_US-Device R?
-U 1 1 610191AF
-P 6400 2500
-AR Path="/610191AF" Ref="R?"  Part="1"
-AR Path="/6100EEBD/610191AF" Ref="R7"  Part="1"
-F 0 "R7" V 6500 2500 50  0000 C CNN
-F 1 "100k" V 6600 2500 50  0000 C CNN
-F 2 "" V 6440 2490 50  0001 C CNN
-F 3 "~" H 6400 2500 50  0001 C CNN
-	1    6400 2500
-	0    1    1    0
-$EndComp
-$Comp
-L Franzininho-Wearable-rescue:R_US-Device R?
-U 1 1 610191A9
-P 6400 2300
-AR Path="/610191A9" Ref="R?"  Part="1"
-AR Path="/6100EEBD/610191A9" Ref="R6"  Part="1"
-F 0 "R6" V 6195 2300 50  0000 C CNN
-F 1 "80k" V 6286 2300 50  0000 C CNN
-F 2 "" V 6440 2290 50  0001 C CNN
-F 3 "~" H 6400 2300 50  0001 C CNN
-	1    6400 2300
-	0    1    1    0
-$EndComp
 Text HLabel 7000 4400 2    50   Output ~ 0
 OUT
@@
 Wire Wire Line
 	4450 4300 4700 4300
-Connection ~ 6650 3800
-Wire Wire Line
-	6650 3450 6650 3800
 Connection ~ 5600 3800
 Wire Wire Line
 	5600 3450 5600 3800
-$Comp
-L Franzininho-Wearable-rescue:C_Small-Device C?
-U 1 1 61019233
-P 6150 3450
-AR Path="/61019233" Ref="C?"  Part="1"
-AR Path="/6100EEBD/61019233" Ref="C5"  Part="1"
-F 0 "C5" V 5921 3450 50  0000 C CNN
-F 1 "100n" V 6012 3450 50  0000 C CNN
-F 2 "" H 6150 3450 50  0001 C CNN
-F 3 "~" H 6150 3450 50  0001 C CNN
-	1    6150 3450
-	0    1    1    0
-$EndComp
-$Comp
-L Franzininho-Wearable-rescue:R_US-Device R?
-U 1 1 6101922D
-P 6150 3800
-AR Path="/6101922D" Ref="R?"  Part="1"
-AR Path="/6100EEBD/6101922D" Ref="R5"  Part="1"
-F 0 "R5" V 5945 3800 50  0000 C CNN
-F 1 "1M" V 6036 3800 50  0000 C CNN
-F 2 "" V 6190 3790 50  0001 C CNN
-F 3 "~" H 6150 3800 50  0001 C CNN
-	1    6150 3800
-	0    1    1    0
-$EndComp
 Wire Wire Line
 	5750 4500 5500 4500
 Wire Wire Line
-	6650 3800 6650 4400
-Wire Wire Line
-	6300 3800 6650 3800
-Wire Wire Line
 	5600 3800 5600 4300
 Wire Wire Line
 	6000 3800 5600 3800
 Wire Wire Line
-	6250 3450 6650 3450
-Wire Wire Line
-	5600 3450 6050 3450
-Wire Wire Line
-	6650 4400 7000 4400
-Connection ~ 6650 4400
-Wire Wire Line
-	6550 4400 6650 4400
+	5600 3450 6000 3450
 Wire Wire Line
 	5600 4300 5750 4300
 Connection ~ 5600 4300
-Wire Wire Line
-	5450 4300 5600 4300
-Wire Wire Line
-	5000 4300 5250 4300
-$Comp
-L Franzininho-Wearable-rescue:R_US-Device R?
-U 1 1 610191FF
-P 4850 4300
-AR Path="/610191FF" Ref="R?"  Part="1"
-AR Path="/6100EEBD/610191FF" Ref="R3"  Part="1"
-F 0 "R3" V 4645 4300 50  0000 C CNN
-F 1 "1k" V 4736 4300 50  0000 C CNN
-F 2 "" V 4890 4290 50  0001 C CNN
-F 3 "~" H 4850 4300 50  0001 C CNN
-	1    4850 4300
-	0    1    1    0
-$EndComp
-$Comp
-L Franzininho-Wearable-rescue:LM324N_NOPB-LM324N_NOPB U?
+$Comp
+L Franzininho_Wearable_SchLib:LM324N_NOPB U?
 U 3 1 610191EF
 P 6150 4400
@@
 	1    0    0    -1
 $EndComp
-$Comp
-L Franzininho-Wearable-rescue:C_Small-Device C?
-U 1 1 610191E5
-P 5350 4300
-AR Path="/610191E5" Ref="C?"  Part="1"
-AR Path="/6100EEBD/610191E5" Ref="C1"  Part="1"
-F 0 "C1" V 5121 4300 50  0000 C CNN
-F 1 "47u" V 5212 4300 50  0000 C CNN
-F 2 "" H 5350 4300 50  0001 C CNN
-F 3 "~" H 5350 4300 50  0001 C CNN
-	1    5350 4300
-	0    1    1    0
-$EndComp
+Connection ~ 6650 4400
+Wire Wire Line
+	6550 4400 6650 4400
+Wire Wire Line
+	6650 4400 7000 4400
+Wire Wire Line
+	6300 3800 6650 3800
+Wire Wire Line
+	6650 3800 6650 4400
+Wire Wire Line
+	6650 3450 6650 3800
+Connection ~ 6650 3800
+$Comp
+L Device:R R1
+U 1 1 61061081
+P 4850 2200
+F 0 "R1" V 4643 2200 50  0000 C CNN
+F 1 "82k" V 4734 2200 50  0000 C CNN
+F 2 "" V 4780 2200 50  0001 C CNN
+F 3 "~" H 4850 2200 50  0001 C CNN
+	1    4850 2200
+	0    1    1    0
+$EndComp
+$Comp
+L Device:R R2
+U 1 1 61063E8E
+P 4850 2400
+F 0 "R2" V 4950 2400 50  0000 C CNN
+F 1 "100k" V 5050 2400 50  0000 C CNN
+F 2 "" V 4780 2400 50  0001 C CNN
+F 3 "~" H 4850 2400 50  0001 C CNN
+	1    4850 2400
+	0    1    1    0
+$EndComp
+$Comp
+L Device:R R4
+U 1 1 6106410B
+P 5450 1600
+F 0 "R4" V 5243 1600 50  0000 C CNN
+F 1 "10k" V 5334 1600 50  0000 C CNN
+F 2 "" V 5380 1600 50  0001 C CNN
+F 3 "~" H 5450 1600 50  0001 C CNN
+	1    5450 1600
+	0    1    1    0
+$EndComp
+$Comp
+L Device:R R6
+U 1 1 61064484
+P 6400 2300
+F 0 "R6" V 6193 2300 50  0000 C CNN
+F 1 "82k" V 6284 2300 50  0000 C CNN
+F 2 "" V 6330 2300 50  0001 C CNN
+F 3 "~" H 6400 2300 50  0001 C CNN
+	1    6400 2300
+	0    1    1    0
+$EndComp
+$Comp
+L Device:R R7
+U 1 1 610648EA
+P 6400 2500
+F 0 "R7" V 6500 2500 50  0000 C CNN
+F 1 "100k" V 6600 2500 50  0000 C CNN
+F 2 "" V 6330 2500 50  0001 C CNN
+F 3 "~" H 6400 2500 50  0001 C CNN
+	1    6400 2500
+	0    1    1    0
+$EndComp
+$Comp
+L Device:R R5
+U 1 1 61065525
+P 6150 3800
+F 0 "R5" V 5950 3800 50  0000 C CNN
+F 1 "1M" V 6050 3800 50  0000 C CNN
+F 2 "" V 6080 3800 50  0001 C CNN
+F 3 "~" H 6150 3800 50  0001 C CNN
+	1    6150 3800
+	0    1    1    0
+$EndComp
+$Comp
+L Device:R R8
+U 1 1 610659CD
+P 6800 5750
+F 0 "R8" V 6900 5750 50  0000 C CNN
+F 1 "100k" V 7000 5750 50  0000 C CNN
+F 2 "" V 6730 5750 50  0001 C CNN
+F 3 "~" H 6800 5750 50  0001 C CNN
+	1    6800 5750
+	0    1    1    0
+$EndComp
+$Comp
+L Device:C C6
+U 1 1 61065F7C
+P 6150 3450
+F 0 "C6" V 5898 3450 50  0000 C CNN
+F 1 "100n" V 5989 3450 50  0000 C CNN
+F 2 "" H 6188 3300 50  0001 C CNN
+F 3 "~" H 6150 3450 50  0001 C CNN
+	1    6150 3450
+	0    1    1    0
+$EndComp
+Wire Wire Line
+	6300 3450 6650 3450
+Wire Wire Line
+	5450 4300 5600 4300
+Wire Wire Line
+	5000 4300 5150 4300
+$Comp
+L Device:C C5
+U 1 1 61066AF3
+P 5300 4300
+F 0 "C5" V 5048 4300 50  0000 C CNN
+F 1 "47u" V 5139 4300 50  0000 C CNN
+F 2 "" H 5338 4150 50  0001 C CNN
+F 3 "~" H 5300 4300 50  0001 C CNN
+	1    5300 4300
+	0    1    1    0
+$EndComp
+$Comp
+L Device:R R3
+U 1 1 61064E83
+P 4850 4300
+F 0 "R3" V 4650 4300 50  0000 C CNN
+F 1 "1k" V 4750 4300 50  0000 C CNN
+F 2 "" V 4780 4300 50  0001 C CNN
+F 3 "~" H 4850 4300 50  0001 C CNN
+	1    4850 4300
+	0    1    1    0
+$EndComp
