File: Franzininho Wearable/Power.sch (KiCad schematic (older format))
At the start: 5 parts, among them U1 ICL7660SCPAZ

Commit message: Correção das bibliotecas de simbolos
Parts:
- removed C11, C4: 10u, symbol Franzininho-Wearable-rescue:CP1-Device
- removed C2, C3: 100n, symbol Franzininho-Wearable-rescue:C_Small-Device
- added C1, C2: 100n, symbol Device:C
- added C3, C4: 10u, symbol Device:CP1
- U1: symbol ICL7660SCPAZ:ICL7660SCPAZ -> Franzininho_Wearable_SchLib:ICL7660SCPAZ
Connections:
- net labels removed: PWR
Changed lines of the file:
@@
 Comment4 ""
 $EndDescr
-$Comp
-L Franzininho-Wearable-rescue:CP1-Device C?
-U 1 1 60FF9720
-P 4950 3850
-AR Path="/60FF9720" Ref="C?"  Part="1"
-AR Path="/60FED1B2/60FF9720" Ref="C11"  Part="1"
-F 0 "C11" H 4650 3900 50  0000 L CNN
-F 1 "10u" H 4650 3800 50  0000 L CNN
-F 2 "" H 4950 3850 50  0001 C CNN
-F 3 "~" H 4950 3850 50  0001 C CNN
-	1    4950 3850
-	1    0    0    -1
-$EndComp
 NoConn ~ 5450 3950
 NoConn ~ 5450 3550
 NoConn ~ 5450 4150
-$Comp
-L Franzininho-Wearable-rescue:CP1-Device C?
-U 1 1 60FF9732
-P 7000 3600
-AR Path="/60FF9732" Ref="C?"  Part="1"
-AR Path="/60FED1B2/60FF9732" Ref="C4"  Part="1"
-F 0 "C4" H 7115 3646 50  0000 L CNN
-F 1 "10u" H 7115 3555 50  0000 L CNN
-F 2 "" H 7000 3600 50  0001 C CNN
-F 3 "~" H 7000 3600 50  0001 C CNN
-	1    7000 3600
-	1    0    0    -1
-$EndComp
 Wire Wire Line
 	5450 3750 5250 3750
@@
 Wire Wire Line
 	4950 4050 4950 4000
-$Comp
-L Franzininho-Wearable-rescue:C_Small-Device C2
-U 1 1 60FF9747
-P 2400 3050
-F 0 "C2" H 2492 3096 50  0000 L CNN
-F 1 "100n" H 2492 3005 50  0000 L CNN
-F 2 "" H 2400 3050 50  0001 C CNN
-F 3 "~" H 2400 3050 50  0001 C CNN
-	1    2400 3050
-	1    0    0    -1
-$EndComp
-$Comp
-L Franzininho-Wearable-rescue:C_Small-Device C3
-U 1 1 60FF974D
-P 2900 3050
-F 0 "C3" H 2992 3096 50  0000 L CNN
-F 1 "100n" H 2992 3005 50  0000 L CNN
-F 2 "" H 2900 3050 50  0001 C CNN
-F 3 "~" H 2900 3050 50  0001 C CNN
-	1    2900 3050
-	1    0    0    -1
-$EndComp
 Wire Wire Line
 	2400 2800 2400 2950
@@
 	2900 2800 2900 2950
 Wire Wire Line
-	2300 3300 2400 3300
+	2300 3400 2400 3400
 Wire Wire Line
-	2900 3150 2900 3300
+	2900 3250 2900 3400
 Wire Wire Line
-	2400 3150 2400 3300
-Connection ~ 2400 3300
+	2400 3250 2400 3400
+Connection ~ 2400 3400
 Wire Wire Line
-	2400 3300 2900 3300
+	2400 3400 2900 3400
 Wire Wire Line
 	2350 2800 2400 2800
@@
 -BATT
 $Comp
-L ICL7660SCPAZ:ICL7660SCPAZ U1
+L Franzininho_Wearable_SchLib:ICL7660SCPAZ U1
 U 1 1 60FF976F
 P 6150 3750
@@
 Text HLabel 2350 2800 0    50   Output ~ 0
 +BATT
-Text HLabel 2300 3300 0    50   Output ~ 0
+Text HLabel 2300 3400 0    50   Output ~ 0
 GND
 Text HLabel 7100 3850 2    50   Output ~ 0
@@
 	2900 2750 2900 2800
 $Comp
-L Franzininho-Wearable-rescue:PWR #PWR?
-U 1 1 61067E48
+L Device:CP1 C3
+U 1 1 6105A28D
+P 4950 3850
+F 0 "C3" H 5065 3896 50  0000 L CNN
+F 1 "10u" H 5065 3805 50  0000 L CNN
+F 2 "" H 4950 3850 50  0001 C CNN
+F 3 "~" H 4950 3850 50  0001 C CNN
+	1    4950 3850
+	1    0    0    -1
+$EndComp
+$Comp
+L Device:CP1 C4
+U 1 1 6105B364
+P 7000 3600
+F 0 "C4" H 7115 3646 50  0000 L CNN
+F 1 "10u" H 7115 3555 50  0000 L CNN
+F 2 "" H 7000 3600 50  0001 C CNN
+F 3 "~" H 7000 3600 50  0001 C CNN
+	1    7000 3600
+	1    0    0    -1
+$EndComp
+$Comp
+L power:+BATT #PWR01
+U 1 1 6105D25B
 P 2400 2750
-AR Path="/61067E48" Ref="#PWR?"  Part="1"
-AR Path="/60FED1B2/61067E48" Ref="#PWR0104"  Part="1"
-F 0 "#PWR0104" H 2400 2600 50  0001 C CNN
-F 1 "PWR" H 2415 2923 50  0001 C CNN
+F 0 "#PWR01" H 2400 2600 50  0001 C CNN
+F 1 "+BATT" H 2415 2923 50  0000 C CNN
 F 2 "" H 2400 2750 50  0001 C CNN
 F 3 "" H 2400 2750 50  0001 C CNN
@@
 $EndComp
 $Comp
-L Franzininho-Wearable-rescue:PWR #PWR?
-U 1 1 6106783D
+L power:-BATT #PWR02
+U 1 1 6105D9E8
 P 2900 2750
-AR Path="/6106783D" Ref="#PWR?"  Part="1"
-AR Path="/60FED1B2/6106783D" Ref="#PWR0103"  Part="1"
-F 0 "#PWR0103" H 2900 2600 50  0001 C CNN
-F 1 "PWR" H 2915 2923 50  0001 C CNN
+F 0 "#PWR02" H 2900 2600 50  0001 C CNN
+F 1 "-BATT" H 2915 2923 50  0000 C CNN
 F 2 "" H 2900 2750 50  0001 C CNN
 F 3 "" H 2900 2750 50  0001 C CNN
@@
 	1    0    0    -1
 $EndComp
+$Comp
+L Device:C C1
+U 1 1 61068DC1
+P 2400 3100
+F 0 "C1" H 2515 3146 50  0000 L CNN
+F 1 "100n" H 2515 3055 50  0000 L CNN
+F 2 "" H 2438 2950 50  0001 C CNN
+F 3 "~" H 2400 3100 50  0001 C CNN
+	1    2400 3100
+	1    0    0    -1
+$EndComp
+$Comp
+L Device:C C2
+U 1 1 610693CB
+P 2900 3100
+F 0 "C2" H 3015 3146 50  0000 L CNN
+F 1 "100n" H 3015 3055 50  0000 L CNN
+F 2 "" H 2938 2950 50  0001 C CNN
+F 3 "~" H 2900 3100 50  0001 C CNN
+	1    2900 3100
+	1    0    0    -1
+$EndComp
